File: BenchBudEE.kicad_pcb (KiCad board)
At the start: 4 copper layers, 165.1 x 63.5 mm, 70 parts, among them K1 1461069-5, P1 24 pin MiniFit JR, P2 CONN_2, P3 CONN_3X2, P4 12 Pin Terminal Block, P5 3 Pin TB, Q1 1461069-5, U1 6N137S-TA1, U10 MCP3901, U11 LMT84, U2 AP5726, U3 MCP4922-E/P, U4 OPA4170, U9 LM324

Commit message: 5.7 Video 2/2 Associating and Placing the Arduino Module
Parts:
- added C11: C, SM0805, B.Cu at (222.6, 153.2)
- added C12: C, SM0805, B.Cu at (264.2, 153.9)
- added D4: B130-13-F, SMA, F.Cu at (266.8, 157.5)
- added Q2: DMN65D8L-7, SOT23GDS, F.Cu at (232.0, 152.8)
- added Q3: AOD476, DPAK2, F.Cu at (272.4, 150.1)
- added Q4: AOD476, DPAK2, F.Cu at (264.4, 150.4)
- added R10: R, SM1206, B.Cu at (272.9, 144.5)
- added R9: R, SM0805, B.Cu at (228.9, 154.3)
- added TH5: MINISMDC050F-2, SM1812, B.Cu at (266.6, 150.2)
- U3: value MCP4922-E/P -> MCP4801; footprint DIP-14__300 -> SO8N
- moved U3 89.5 mm to (222.5, 153.8), turned to 270 degrees
- moved R35 24.6 mm to (302.8, 181.0)
- moved R36 24.5 mm to (306.6, 181.0)
- moved R32 24.5 mm to (314.1, 181.0)
- moved R37 24.5 mm to (310.3, 181.0)
- moved R15 19.6 mm to (202.1, 146.2)
- moved R16 19.6 mm to (172.6, 109.1)
- moved R20 19.6 mm to (182.8, 109.1)
- moved R22 19.6 mm to (191.9, 109.1)
- moved uC1 19.6 mm to (175.6, 128.0)
- moved R11 19.6 mm to (189.4, 146.2)
- moved R12 19.6 mm to (194.4, 146.2)
- moved R13 19.6 mm to (197.0, 146.2)
- moved R14 19.6 mm to (199.5, 146.2)
- moved R17 19.6 mm to (175.1, 109.1)
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Connections:
- net /Arduino/ADC_CS_N renamed /Arduino/~ADC_CS
- U3 pad 1: (no net) -> +5V
- U3 pad 2: (no net) -> /Fan/CS_N
- U3 pad 3: /Fan/CS_N -> /Arduino/SCLK
- U3 pad 4: /Arduino/SCLK -> /Arduino/MOSI
- U3 pad 5: /Arduino/MOSI -> /Arduino/~LDAC
- U3 pad 6: (no net) -> /Arduino/~SHDN
- U3 pad 7: (no net) -> AGND
- U3 pad 8: (no net) -> N-00000122
- uC1 pad 13: (no net) -> N-0000052
- uC1 pad 14: (no net) -> N-0000053

Commit message: 5.8 Associating and Placing the Power Protection and Filtering Module
Parts:
- added C1: C, SM1206, F.Cu at (159.3, 122.3)
- added C13: C, SM1206, F.Cu at (160.8, 142.7)
- added C2: C, SM1206, F.Cu at (159.3, 109.0)
- added L1: CM322522-220KL, SM1210L, F.Cu at (159.3, 117.5)
- added L2: CM322522-220KL, SM1210L, F.Cu at (161.2, 147.8)
- added L3: CM322522-220KL, SM1210L, F.Cu at (159.3, 113.2)
- added R7: R, SM0805, F.Cu at (160.3, 153.5)
- added SW1: Power Switch, BB_Switch, F.Cu at (157.2, 158.1)
- added TH1: THERMISTOR, SM1812, B.Cu at (140.7, 147.1)
- added TH2: THERMISTOR, SM1812, B.Cu at (140.6, 130.0)
- added TH3: THERMISTOR, SM1812, B.Cu at (140.6, 113.4)
- added TH4: THERMISTOR, SM1812, F.Cu at (161.2, 147.8)
- R27: moved to B.Cu
- moved R35 148.8 mm to (373.5, 50.0)
- moved R32 147.4 mm to (372.1, 45.5)
- moved R36 146.9 mm to (378.5, 52.8)
- moved R33 145.1 mm to (376.7, 46.5)
- moved R37 141.3 mm to (379.7, 57.9)
- moved U9 140.6 mm to (373.5, 41.7)
- moved R28 137.6 mm to (367.3, 52.2)
- moved R29 131.3 mm to (373.6, 55.6)
- moved R31 130.1 mm to (365.6, 48.4)
- moved U2 129.2 mm to (363.5, 41.3)
- moved R30 127.6 mm to (367.0, 58.5)
- moved R34 125.6 mm to (374.4, 60.6)
- moved R27 105.7 mm to (252.3, 99.1), turned to 90 degrees

Commit message: 5.10 Video 2/2 Associating and Placing the Power Modification Module
Parts:
- added C14: C, SM0805, B.Cu at (177.2, 135.8)
- added C15: C, SM0805, B.Cu at (179.8, 112.3)
- added C16: C, SM0805, B.Cu at (220.6, 112.3)
- added C17: C, SM0805, B.Cu at (219.3, 134.4)
- added C18: C, SM0805, B.Cu at (220.6, 117.3)
- added C19: C, SM0805, B.Cu at (219.5, 139.4)
- added C20: C, SM0805, B.Cu at (181.0, 134.1)
- added C21: C, SM0805, B.Cu at (176.4, 114.9)
- added C22: C, SM0805, B.Cu at (219.3, 136.9)
- added C23: C, SM0805, B.Cu at (181.1, 136.7)
- added C24: C, SM0805, B.Cu at (191.4, 114.3)
- added C25: C, SM0805, B.Cu at (214.4, 132.5)
- added D10: MMBD914-7-F, SOT23_DIODE, B.Cu at (186.7, 138.6)
- added D11: MMBD914-7-F, SOT23_DIODE, F.Cu at (226.3, 114.8)
- added D12: MMBD914-7-F, SOT23_DIODE, F.Cu at (187.5, 112.1)
- added D5: MMBD914-7-F, SOT23_DIODE, B.Cu at (226.4, 136.4)
- added D6: MMBD914-7-F, SOT23_DIODE, F.Cu at (190.6, 138.2)
- added D7: MMBD914-7-F, SOT23_DIODE, B.Cu at (186.7, 116.3)
- added D8: MMBD914-7-F, SOT23_DIODE, B.Cu at (230.0, 114.8)
- added D9: MMBD914-7-F, SOT23_DIODE, B.Cu at (228.6, 136.7)
- added R52: R, SM0805_blob, F.Cu at (199.5, 106.6)
- added R53: R, SM0805_blob, F.Cu at (202.1, 106.6)
- added R54: R, SM0805, B.Cu at (177.3, 137.8)
- added R55: R, SM0805, B.Cu at (181.0, 139.4)
- added U5: LM317K, TO220, F.Cu at (211.1, 136.9)
- added U6: LM337T, TO220, F.Cu at (212.5, 114.9)
- added U7: LM337T, TO220, F.Cu at (171.8, 114.9)
- added U8: LM317, TO220, F.Cu at (172.6, 136.7)
- R28: value RVAR -> 5K; footprint SM0805 -> EVUE3K
- R29, R30: value R -> 715; moved to B.Cu
- R31: value RVAR -> 5k; footprint SM0805 -> EVUE3K
- R32, R33, R34, R35, R36, R37: moved to B.Cu
- moved R33 208.4 mm to (179.8, 114.9), turned to 180 degrees
- moved R32 205.3 mm to (179.8, 117.5)
- moved R35 201.5 mm to (190.0, 133.2), turned to 180 degrees
- moved R36 198.2 mm to (191.1, 117.6), turned to 180 degrees
- moved R28 177.0 mm to (225.8, 158.5), turned to 270 degrees
- moved R29 176.4 mm to (219.6, 141.6)
- moved R34 170.8 mm to (219.3, 132.1)
- moved R37 169.0 mm to (220.6, 114.9)
- moved R30 158.8 mm to (220.6, 119.9)
- moved R31 148.4 mm to (225.3, 96.6), turned to 90 degrees
- moved U9 87.4 mm to (334.5, 119.9)
- moved U2 83.1 mm to (327.5, 116.2)
- moved P2 21.6 mm to (237.6, 140.5)
- moved U3 21.0 mm to (243.5, 154.6)
- moved C11 20.7 mm to (243.2, 154.9)
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Connections:
- R28 pad 1: N-00000133 -> N-00000137
- R28 pad 2: N-00000140 -> AGND
- R29 pad 1: AGND -> N-00000137
- R29 pad 2: N-00000140 -> /PowerAdjustmentMonitor/V+_ADJ
- R30 pad 1: AGND -> N-00000141
- R30 pad 2: N-00000127 -> /PowerAdjustmentMonitor/V-_ADJ
- R31 pad 1: N-00000127 -> N-00000141
- R31 pad 2: N-00000135 -> N-00000131
- R32 pad 1: N-00000135 -> AGND
- R32 pad 2: /PowerAdjustmentMonitor/V-_ADJ -> N-00000140
- R33 pad 1: N-00000133 -> N-00000140
- R33 pad 2: /PowerAdjustmentMonitor/V+_ADJ -> FE_V-
- R37 pad 2: (no net) -> /PowerAdjustmentMonitor/V-_ADJ

Commit message: 5.11 Video 2/2 Associating and Placing the LED Driver Module
Parts:
- removed U9: LM324, SOT323
- added C3: 1uF, SM0805, B.Cu at (220.3, 126.0)
- added C4: 1uF, SM0805, B.Cu at (222.6, 126.0)
- added D3: B0540WS-7, SOD-323, F.Cu at (220.0, 127.3)
- added L4: 22uH, NR4012, F.Cu at (226.7, 124.6)
- added R8: 15, SM0805, B.Cu at (225.4, 126.0)
- U2: footprint SSOP20 -> SOT23_6
- moved U2 105.1 mm to (222.9, 126.0)
- moved D9 10.2 mm to (228.7, 146.8)
- moved C19 10.2 mm to (219.6, 149.6)
- moved D5 10.2 mm to (226.6, 146.6)
- moved R29 10.2 mm to (219.7, 151.8)
- moved C17 10.2 mm to (219.5, 144.5)
- moved C22 10.2 mm to (219.5, 147.1)
- moved C25 10.2 mm to (214.5, 142.6)
- moved R34 10.2 mm to (219.5, 142.2)
- moved U5 9.53 mm to (211.3, 146.4)
- moved D11 7.03 mm to (225.6, 107.8)
- moved D8 7.03 mm to (229.2, 107.8)
- moved C16 7.03 mm to (219.8, 105.3)
- moved C18 7.03 mm to (219.8, 110.4)
- moved R30 7.03 mm to (219.8, 112.9)
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
Commit message: 5.13 Video 1/2 @ 12m:30s  Finalizing The System Part Placement
Parts:
- moved D3 55.0 mm to (274.7, 132.8)
- moved L4 55.0 mm to (281.4, 130.2)
- moved U2 55.0 mm to (277.6, 131.6)
- moved C3 55.0 mm to (275.1, 131.6)
- moved C4 55.0 mm to (277.4, 131.6)
- moved R8 55.0 mm to (280.2, 131.6)
- moved P5 47.0 mm to (296.9, 158.1)
- moved R3 46.7 mm to (267.3, 162.7)
- moved R4 46.7 mm to (264.2, 149.9)
- moved R5 46.7 mm to (262.9, 162.7)
- moved D1 46.7 mm to (263.8, 156.2)
- moved D2 46.7 mm to (258.6, 160.7)
- moved K1 46.7 mm to (269.6, 157.7)
- moved R2 46.7 mm to (262.9, 160.3)
- moved Q1 46.7 mm to (267.0, 159.4)
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Changed lines of the file:
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@@
     (links 322)
     (no_connects 232)
-    (area 134.315999 96.850999 299.516001 160.451001)
+    (area 133.405999 72.303999 300.253517 185.125001)
     (thickness 1.6)
     (drawings 4)
@@
   )
   (module TE-SPDT (layer F.Cu)
-    (at 269.621 110.998)
+    (at 269.621 157.734)
     (fp_text reference K1 (at 4.572 -16.256) (layer F.SilkS)
       (effects (font (size 1 1) (thickness 0.15)))
@@
   )
   (module SOT23 (layer B.Cu)
-    (at 266.954 112.649 180)
+    (at 266.954 159.385 180)
     (tags SOT23)
     (fp_text reference Q1 (at 1.99898 0.09906 450) (layer B.SilkS)
@@
   )
   (module SMA (layer F.Cu)
-    (at 258.572 113.919 90)
+    (at 258.572 160.655 90)
     (fp_text reference D2 (at 2.54 -3.81 90) (layer F.SilkS)
       (effects (font (size 1 1) (thickness 0.15)))
@@
   )
   (module SM0805 (layer B.Cu)
-    (at 262.89 115.951 180)
+    (at 262.89 162.687 180)
     (attr smd)
     (fp_text reference R5 (at 0 0.3175 180) (layer B.SilkS)
@@
   )
   (module SM0805 (layer B.Cu)
-    (at 274.447 99.822 90)
+    (at 274.447 146.558 90)
     (attr smd)
     (fp_text reference R6 (at 0 0.3175 90) (layer B.SilkS)
@@
   )
   (module SM0805 (layer B.Cu)
-    (at 254.635 99.06 270)
+    (at 254.635 145.796 270)
     (attr smd)
     (fp_text reference R1 (at 0 0.3175 270) (layer B.SilkS)
@@
   )
   (module SM0805 (layer B.Cu)
-    (at 264.16 103.124 180)
+    (at 264.16 149.86 180)
     (attr smd)
     (fp_text reference R4 (at 0 0.3175 180) (layer B.SilkS)
@@
   )
   (module SM0805 (layer B.Cu)
-    (at 262.89 113.538 180)
+    (at 262.89 160.274 180)
     (attr smd)
     (fp_text reference R2 (at 0 0.3175 180) (layer B.SilkS)
@@
   )
   (module SM0805 (layer B.Cu)
-    (at 267.335 115.951 180)
+    (at 267.335 162.687 180)
     (attr smd)
     (fp_text reference R3 (at 0 0.3175 180) (layer B.SilkS)
@@
   )
   (module LED-0805 (layer F.Cu)
-    (at 263.779 109.474)
+    (at 263.779 156.21)
     (descr "LED 0805 smd package")
     (tags "LED 0805 SMD")
@@
   )
   (module 8-SMD (layer F.Cu)
-    (at 257.175 107.315)
+    (at 257.175 154.051)
     (fp_text reference U1 (at 3.81 -11.938) (layer F.SilkS)
       (effects (font (size 1 1) (thickness 0.15)))
@@
   )
   (module SOT353 (layer F.Cu)
-    (at 284.226 150.876)
+    (at 287.401 117.475)
     (descr SOT353)
     (attr smd)
@@
   )
   (module SO14N (layer F.Cu)
-    (at 258.064 140.843)
+    (at 262.509 107.696)
     (descr "Module CMS SOJ 14 pins Large")
     (tags "CMS SOJ")
@@
   )
   (module SM1206 (layer B.Cu)
-    (at 257.7465 143.1925 90)
+    (at 262.1915 110.0455 90)
     (attr smd)
     (fp_text reference R40 (at 0 0 90) (layer B.SilkS)
@@
   )
   (module SM1206 (layer B.Cu)
-    (at 254.508 143.256 90)
+    (at 258.953 110.109 90)
     (attr smd)
     (fp_text reference R41 (at 0 0 90) (layer B.SilkS)
@@
   )
   (module SM1206 (layer B.Cu)
-    (at 248.3485 143.256 270)
+    (at 252.7935 110.109 270)
     (attr smd)
     (fp_text reference R39 (at 0 0 270) (layer B.SilkS)
@@
   )
   (module SM1206 (layer B.Cu)
-    (at 251.5235 143.256 270)
+    (at 255.9685 110.109 270)
     (attr smd)
     (fp_text reference R38 (at 0 0 270) (layer B.SilkS)
@@
   )
   (module SM0805 (layer B.Cu)
-    (at 245.5545 148.717 270)
+    (at 249.9995 115.57 270)
     (attr smd)
     (fp_text reference C5 (at 0 0.3175 270) (layer B.SilkS)
@@
   )
   (module SM0805 (layer B.Cu)
-    (at 243.205 148.717 270)
+    (at 247.65 115.57 270)
     (attr smd)
     (fp_text reference C6 (at 0 0.3175 270) (layer B.SilkS)
@@
   )
   (module SM0805 (layer B.Cu)
-    (at 258.191 134.6835 90)
+    (at 262.636 101.5365 90)
     (attr smd)
     (fp_text reference C9 (at 0 0.3175 90) (layer B.SilkS)
@@
   )
   (module SM0805 (layer B.Cu)
-    (at 255.0795 139.446)
+    (at 259.5245 106.299)
     (attr smd)
     (fp_text reference C10 (at 0 0.3175) (layer B.SilkS)
@@
   )
   (module SM0805 (layer B.Cu)
-    (at 248.0945 132.7785 90)
+    (at 252.5395 99.6315 90)
     (attr smd)
     (fp_text reference R46 (at 0 0.3175 90) (layer B.SilkS)
@@
   )
   (module SM0805 (layer B.Cu)
-    (at 245.5545 132.715 90)
+    (at 249.9995 99.568 90)
     (attr smd)
     (fp_text reference R45 (at 0 0.3175 90) (layer B.SilkS)
@@
   )
   (module SM0805 (layer B.Cu)
-    (at 284.226 150.876 90)
+    (at 287.782 117.856 90)
     (attr smd)
     (fp_text reference C7 (at 0 0.3175 90) (layer B.SilkS)
@@
   )
   (module SM0805 (layer F.Cu)
-    (at 242.951 144.78 180)
+    (at 247.396 111.633 180)
     (attr smd)
     (fp_text reference C8 (at 0 -0.3175 180) (layer F.SilkS)
@@
   )
   (module SM0805 (layer B.Cu)
-    (at 261.4295 135.636 180)
+    (at 265.8745 102.489 180)
     (attr smd)
     (fp_text reference R42 (at 0 0.3175 180) (layer B.SilkS)
@@
   )
   (module pin_array_3x2 (layer F.Cu)
-    (at 245.491 126.365 180)
+    (at 240.665 100.203 180)
     (descr "Double rangee de contacts 2 x 4 pins")
     (tags CONN)
@@
   )
   (module PIN_ARRAY_2X1 (layer F.Cu)
-    (at 237.617 140.462 90)
+    (at 242.062 107.315 90)
     (descr "Connecteurs 2 pins")
     (tags "CONN DEV")
@@
   )
   (module SSOP20 (layer F.Cu)
-    (at 242.824 142.875 90)
+    (at 247.269 109.728 90)
     (descr "SSOP 20 pins")
     (tags "CMS SSOP SMD")
@@
   )
   (module SM0805 (layer B.Cu)
-    (at 243.713 142.24 270)
+    (at 248.158 109.093 270)
     (attr smd)
     (fp_text reference R47 (at 0 0.3175 270) (layer B.SilkS)
@@
   )
   (module SM0805 (layer B.Cu)
-    (at 284.226 148.082)
+    (at 287.147 114.935)
     (attr smd)
     (fp_text reference R48 (at 0 0.3175) (layer B.SilkS)
@@
   )
   (module SM0805 (layer B.Cu)
-    (at 242.951 132.7785 90)
+    (at 247.396 99.6315 90)
     (attr smd)
     (fp_text reference R44 (at 0 0.3175 90) (layer B.SilkS)
@@
   )
   (module SM0805 (layer B.Cu)
-    (at 254.762 135.763 180)
+    (at 259.207 102.616 180)
     (attr smd)
     (fp_text reference R43 (at 0 0.3175 180) (layer B.SilkS)
@@
   )
   (module 3pinPhoenixTerminalBlock (layer F.Cu)
-    (at 296.799 111.125 90)
+    (at 296.926 158.115 90)
     (fp_text reference P5 (at 12.319 1.397 90) (layer F.SilkS)
       (effects (font (size 1 1) (thickness 0.15)))
@@
   )
   (module 12pinPhoenixConnector (layer F.Cu)
-    (at 294.386 157.861 90)
+    (at 294.513 141.351 90)
     (fp_text reference P4 (at 42.545 3.175 90) (layer F.SilkS)
       (effects (font (size 1 1) (thickness 0.15)))
@@
   )
   (module SM0805 (layer B.Cu)
-    (at 252.349 99.06 90)
+    (at 252.349 145.796 90)
     (attr smd)
     (fp_text reference R27 (at 0 0.3175 90) (layer B.SilkS)
@@
   )
   (module SOT23GDS (layer F.Cu)
-    (at 252.603 154.559)
+    (at 257.048 121.412)
     (descr "Module CMS SOT23 Transistore EBC")
     (tags "CMS SOT")
@@
   )
   (module SMA (layer F.Cu)
-    (at 271.907 149.352)
+    (at 276.352 116.205)
     (fp_text reference D4 (at 2.54 -3.81) (layer F.SilkS)
       (effects (font (size 1 1) (thickness 0.15)))
@@
   )
   (module SM1812 (layer B.Cu)
-    (at 271.653 142.113)
+    (at 276.098 108.966)
     (tags "CMS SM")
     (attr smd)
@@
   )
   (module SM1206 (layer B.Cu)
-    (at 278.003 136.398)
+    (at 282.448 103.251)
     (attr smd)
     (fp_text reference R10 (at 0 0) (layer B.SilkS)
@@
   )
   (module SM0805 (layer B.Cu)
-    (at 249.428 156.083 180)
+    (at 253.873 122.936 180)
     (attr smd)
     (fp_text reference R9 (at 0 0.3175 180) (layer B.SilkS)
@@
   )
   (module SO8N (layer F.Cu)
-    (at 243.459 154.559 270)
+    (at 247.904 121.412 270)
     (descr "Module CMS SOJ 8 pins large")
     (tags "CMS SOJ")
@@
   )
   (module SM0805 (layer B.Cu)
-    (at 269.24 145.796)
+    (at 273.685 112.649)
     (attr smd)
     (fp_text reference C12 (at 0 0.3175) (layer B.SilkS)
@@
   )
   (module SM0805 (layer B.Cu)
-    (at 243.205 154.94 270)
+    (at 247.65 121.793 270)
     (attr smd)
     (fp_text reference C11 (at 0 0.3175 270) (layer B.SilkS)
@@
   )
   (module DPAK2 (layer F.Cu)
-    (at 269.494 142.24)
+    (at 273.939 109.093)
     (descr "MOS boitier DPACK G-D-S")
     (tags "CMD DPACK")
@@
   )
   (module DPAK2 (layer F.Cu)
-    (at 277.495 141.986)
+    (at 281.94 108.839)
     (descr "MOS boitier DPACK G-D-S")
     (tags "CMD DPACK")
@@
   )
   (module SOD-323 (layer F.Cu)
-    (at 219.964 127.254 90)
+    (at 274.701 132.842 90)
     (fp_text reference D3 (at 1.5 -3.1 90) (layer F.SilkS)
       (effects (font (size 1 1) (thickness 0.15)))
@@
   )
   (module SM0805 (layer B.Cu)
-    (at 220.345 125.984 270)
+    (at 275.082 131.572 270)
     (attr smd)
     (fp_text reference C3 (at 0 0.3175 270) (layer B.SilkS)
@@
   )
   (module SM0805 (layer B.Cu)
-    (at 222.631 125.984 270)
+    (at 277.368 131.572 270)
     (attr smd)
     (fp_text reference C4 (at 0 0.3175 270) (layer B.SilkS)
@@
   )
   (module SM0805 (layer B.Cu)
-    (at 225.425 125.984 270)
+    (at 280.162 131.572 270)
     (attr smd)
     (fp_text reference R8 (at 0 0.3175 270) (layer B.SilkS)
@@
   )
   (module NR4012 (layer F.Cu)
-    (at 226.695 124.587 270)
+    (at 281.432 130.175 270)
     (fp_text reference L4 (at 1.4 -3.3 270) (layer F.SilkS)
       (effects (font (size 1 1) (thickness 0.15)))
@@
   )
   (module SOT23_6 (layer F.Cu)
-    (at 222.885 125.984)
+    (at 277.622 131.572)
     (fp_text reference U2 (at 1.99898 0 90) (layer F.SilkS)
       (effects (font (size 0.762 0.762) (thickness 0.0762)))

Commit message: 5.13 Video 1/2 Finalizing The System Part Placement
Parts:
- moved R31 55.1 mm to (235.7, 152.8), turned to 270 degrees
- moved U6 38.5 mm to (234.4, 140.3), turned to 90 degrees
- moved C16 29.1 mm to (230.5, 132.3), turned to 270 degrees
- moved R37 27.8 mm to (233.2, 132.3), turned to 90 degrees
- moved C18 27.0 mm to (235.6, 132.3), turned to 270 degrees
- moved R30 26.7 mm to (238.1, 132.3), turned to 90 degrees
- moved D9 25.6 mm to (219.6, 122.9), turned to 90 degrees
- moved D5 22.7 mm to (219.3, 125.1), turned to 90 degrees
- moved R29 20.4 mm to (224.5, 132.0), turned to 90 degrees
- moved D11 20.2 mm to (233.0, 126.6), turned to 90 degrees
- moved C19 17.7 mm to (222.4, 132.1), turned to 90 degrees
- moved D8 15.6 mm to (233.0, 122.9), turned to 90 degrees
- moved C22 14.9 mm to (219.8, 132.2), turned to 90 degrees
- moved C17 12.5 mm to (217.3, 132.2), turned to 90 degrees
- moved R34 11.0 mm to (215.0, 132.2), turned to 90 degrees
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